Commit message: Part 2 Sec 6 Done

File: src/car_description/urdf/a_car.urdf.xacro (robot description, xacro)
@@ -3,5 +3,6 @@
     <xacro:include filename="common_properties.xacro" />
     <xacro:include filename="mobile_base.xacro" />
-    <xacro:macro name="example_macro" params="a b c">
+    <xacro:include filename="mobile_base_gazebo.xacro" />
+    <!-- <xacro:macro name="example_macro" params="a b c">
         <link name="dummy_link">
             <visual>
@@ -11,4 +12,4 @@
             </visual>
         </link>
-    </xacro:macro>
+    </xacro:macro> -->
 </robot>

File: src/udemy_robot_description/urdf/mobile_base.xacro (robot description, xacro)
@@ -6,9 +6,5 @@
     <xacro:property name="wheel_radius" value="0.1" />
     <xacro:property name="wheel_length" value="0.05" />
-    <xacro:property name="box_mass" value="5.0" />
-    <xacro:property name="wheel_mass" value="4.0" />
-    <xacro:property name="caster_wheel_mass" value="1.0" />
-    <link name="base_footprint">
-    </link>
+    <link name="base_footprint" />
     <link name="base_link">
         <visual>
@@ -17,5 +13,5 @@
             </geometry>
             <origin xyz="0 0 ${base_height / 2.0}" rpy="0 0 0" />
-            <material name="blue" />
+            <material name="green" />
         </visual>
         <collision>
@@ -25,6 +21,6 @@
             <origin xyz="0 0 ${base_height / 2.0}" rpy="0 0 0" />
         </collision>
-        <xacro:box_inertia m="${box_mass}" l="${base_length}" w="${base_width}" h="${base_height}"
-            xyz="0 0 ${base_height /2.0}" rpy="0 0 0" />
+        <xacro:box_inertia m="5.0" x="${base_length}" y="${base_width}" z="${base_height}"
+                           o_xyz="0 0 ${base_height / 2.0}" o_rpy="0 0 0" />
     </link>
     <xacro:macro name="wheel_link" params="prefix">
@@ -35,14 +31,14 @@
                 </geometry>
                 <origin xyz="0 0 0" rpy="${pi / 2.0} 0 0" />
-                <material name="grey" />
+                <material name="gray" />
             </visual>
             <collision>
                 <geometry>
-                    <cylinder radius="${wheel_radius}" length="${wheel_length}" />
+                    <sphere radius="${wheel_radius}" />
                 </geometry>
-                <origin xyz="0 0 0" rpy="${pi / 2.0} 0 0" />
+                <origin xyz="0 0 0" rpy="0 0 0" />
             </collision>
-            <xacro:cylinder_inertia m="${wheel_mass}" r="${wheel_radius}" h="${wheel_length}"
-                xyz="0 0 0" rpy="${pi / 2.0} 0 0" />
+            <xacro:cylinder_inertia m="1.0" r="${wheel_radius}" l="${wheel_length}"
+                                    o_xyz="0 0 0" o_rpy="${pi / 2.0} 0 0" />
         </link>
     </xacro:macro>
@@ -55,5 +51,5 @@
             </geometry>
             <origin xyz="0 0 0" rpy="0 0 0" />
-            <material name="grey" />
+            <material name="gray" />
         </visual>
         <collision>
@@ -63,11 +59,16 @@
             <origin xyz="0 0 0" rpy="0 0 0" />
         </collision>
-        <xacro:sphere_inertia m="${caster_wheel_mass}" r="${wheel_radius / 2.0}"
-            xyz="0 0 0" rpy="0 0 0" />
+        <xacro:sphere_inertia m="0.5" r="${wheel_radius / 2.0}"
+                              o_xyz="0 0 0" o_rpy="0 0 0" />
     </link>
+    <joint name="base_joint" type="fixed">
+        <parent link="base_footprint" />
+        <child link="base_link" />
+        <origin xyz="0 0 ${wheel_radius}" rpy="0 0 0" />
+    </joint>
     <joint name="base_right_wheel_joint" type="continuous">
         <parent link="base_link" />
         <child link="right_wheel_link" />
-        <origin xyz="-${base_length / 4.0} ${base_width /2.0 + wheel_length/2.0} 0" rpy="0 0 0" />
+        <origin xyz="${-base_length / 4.0} ${-(base_width + wheel_length) / 2.0} 0" rpy="0 0 0" />
         <axis xyz="0 1 0" />
     </joint>
@@ -75,5 +76,5 @@
         <parent link="base_link" />
         <child link="left_wheel_link" />
-        <origin xyz="-${base_length / 4.0} -${base_width / 2.0 + wheel_length/2.0} 0" rpy="0 0 0" />
+        <origin xyz="${-base_length / 4.0} ${(base_width + wheel_length) / 2.0} 0" rpy="0 0 0" />
         <axis xyz="0 1 0" />
     </joint>
@@ -81,10 +82,5 @@
         <parent link="base_link" />
         <child link="caster_wheel_link" />
-        <origin xyz="${base_length / 3.0} 0 -${wheel_radius / 2.0}" rpy="0 0 0" />
-    </joint>
-    <joint name="base_joint" type="fixed">
-        <parent link="base_footprint" />
-        <child link="base_link" />
-        <origin xyz="0 0 ${wheel_radius}" rpy="0 0 0" />
+        <origin xyz="${base_length / 3.0} 0 ${-wheel_radius / 2.0}" rpy="0 0 0" />
     </joint>
 </robot>
