Commit message: Part 2 Sec 6 temp back up

File: src/car_description/urdf/mobile_base.xacro (robot description, xacro)
@@ -6,4 +6,7 @@
     <xacro:property name="wheel_radius" value="0.2" />
     <xacro:property name="wheel_length" value="0.05" />
+    <xacro:property name="box_mass" value="5.0" />
+    <xacro:property name="wheel_mass" value="4.0" />
+    <xacro:property name="caster_wheel_mass" value="1.0" />
     <link name="base_footprint">
     </link>
@@ -16,4 +19,12 @@
             <material name="blue" />
         </visual>
+        <collision>
+            <geometry>
+                <box size="${base_length} ${base_width} ${base_height}" />
+            </geometry>
+            <origin xyz="0 0 ${base_height / 2.0}" rpy="0 0 0" />
+        </collision>
+        <xacro:box_inertia m="${box_mass}" l="${base_length}" w="${base_width}" h="${base_height}"
+            xyz="0 0 ${base_height /2.0}" rpy="0 0 0" />
     </link>
     <xacro:macro name="wheel_link" params="prefix">
@@ -26,4 +37,12 @@
                 <material name="grey" />
             </visual>
+            <collision>
+                <geometry>
+                    <cylinder radius="${wheel_radius}" length="${wheel_length}" />
+                </geometry>
+                <origin xyz="0 0 0" rpy="${pi / 2.0} 0 0" />
+            </collision>
+            <xacro:cylinder_inertia m="${wheel_mass}" r="${wheel_radius}" h="${wheel_length}"
+                xyz="0 0 0" rpy="${pi / 2.0} 0 0" />
         </link>
     </xacro:macro>
@@ -38,4 +57,12 @@
             <material name="grey" />
         </visual>
+        <collision>
+            <geometry>
+                <sphere radius="${wheel_radius / 2.0}" />
+            </geometry>
+            <origin xyz="0 0 0" rpy="0 0 0" />
+        </collision>
+        <xacro:sphere_inertia m="${caster_wheel_mass}" r="${wheel_radius / 2.0}"
+            xyz="0 0 0" rpy="0 0 0" />
     </link>
     <joint name="base_right_wheel_joint" type="continuous">
@@ -57,7 +84,7 @@
     </joint>
     <joint name="base_joint" type="fixed">
-        <parent link="base_link" />
-        <child link="base_footprint" />
-        <origin xyz="0 0 -${wheel_radius}" rpy="0 0 0" />
+        <parent link="base_footprint" />
+        <child link="base_link" />
+        <origin xyz="0 0 ${wheel_radius}" rpy="0 0 0" />
     </joint>
 </robot>

Commit message: Part 2 sect 6 for gazebo old

File: src/car_description/urdf/mobile_base.xacro (robot description, xacro)
@@ -6,5 +6,5 @@
     <xacro:property name="wheel_radius" value="0.1" />
     <xacro:property name="wheel_length" value="0.05" />
-    <xacro:property name="box_mass" value="5.0" />
+    <xacro:property name="box_mass" value="8.0" />
     <xacro:property name="wheel_mass" value="4.0" />
     <xacro:property name="caster_wheel_mass" value="1.0" />

File: src/car_description/urdf/mobile_base_gazebo.xacro (robot description, xacro)
@@ -1,24 +1,35 @@
 <?xml version="1.0"?>
 <robot xmlns:xacro="http://www.ros.org/wiki/xacro">
+    <gazebo reference="base_link">
+        <material>Gazebo/Blue</material>
+    </gazebo>
+    <gazebo reference="right_wheel_link">
+        <material>Gazebo/Grey</material>
+    </gazebo>
+    <gazebo reference="left_wheel_link">
+        <material>Gazebo/Grey</material>
+    </gazebo>
     <gazebo reference="caster_wheel_link">
+        <material>Gazebo/Grey</material>
         <mu1 value="0.1" />
         <mu2 value="0.1" />
     </gazebo>
     <gazebo>
-        <plugin
-            filename="gz-sim-diff-drive-system"
-            name="gz::sim::systems::DiffDrive">
+        <plugin name="gazebo_ros_diff_drive" filename="libgazebo_ros_diff_drive.so">
+            <!-- Update rate in Hz -->
+            <update_rate>50</update_rate>
+            <!-- wheels -->
             <left_joint>base_left_wheel_joint</left_joint>
             <right_joint>base_right_wheel_joint</right_joint>
+            <!-- kinematics -->
             <wheel_separation>0.45</wheel_separation>
-            <wheel_radius>0.1</wheel_radius>
-            <frame_id>odom</frame_id>
-            <child_id_frame>base_footprint</child_id_frame>
-        </plugin>
-    </gazebo>
-    <gazebo>
-        <plugin
-            filename="gz-sim-joint-state-publisher-system"
-            name="gz::sim::systems::JointStatePublisher">
+            <wheel_diameter>0.2</wheel_diameter>
+            <!-- output -->
+            <publish_odom>true</publish_odom>
+            <publish_odom_tf>true</publish_odom_tf>
+            <publish_wheel_tf>true</publish_wheel_tf>
+            <odometry_topic>odom</odometry_topic>
+            <odometry_frame>odom</odometry_frame>
+            <robot_base_frame>base_footprint</robot_base_frame>
         </plugin>
     </gazebo>
