Commit message: Part 2 sec 7 fixed bug

File: src/car_description/urdf/camera.xacro (robot description, xacro)
@@ -10,5 +10,5 @@
                 <box size="${camera_length} ${camera_width} ${camera_height}" />
             </geometry>
-            <material name="grey" />
+            <material name="green" />
         </visual>
         <collision>
@@ -17,12 +17,12 @@
             </geometry>
         </collision>
-        <!-- <xacro:box_inertia m="${camera_mass}"
+        <xacro:box_inertia m="${camera_mass}"
             l="${camera_length}" w="${camera_width}" h="${camera_height}"
-            xyz="0 0 0" rpy="0 0 0" /> -->
+            xyz="0 0 0" rpy="0 0 0" />
     </link>
     <joint name="base_camera_joint" type="fixed">
         <parent link="base_link" />
         <child link="camera_link" />
-        <orgin xyz="0.3 0 ${(base_length + camera_length)/2.0}" rpy="0 0 0" />
+        <origin xyz="${(camera_length+base_length)/2.0} 0 ${camera_height/2.0}" rpy="0 0 0" />
     </joint>
 </robot>

Commit message: Part 2 Sec 7 done

File: src/car_description/urdf/camera.xacro (robot description, xacro)
@@ -26,3 +26,22 @@
         <origin xyz="${(camera_length+base_length)/2.0} 0 ${camera_height/2.0}" rpy="0 0 0" />
     </joint>
+    <!-- open cv -->
+    <link name="camera_optical_link"></link>
+    <joint name="camera_optical_joint" type="fixed">
+        <parent link="camera_link" />
+        <child link="camera_optical_link" />
+        <origin xyz="0 0 0" rpy="${-pi/2.0} 0 ${-pi/2.0}" />
+    </joint>
+    <gazebo reference="camera_link">
+        <material>Gazebo/Green</material>
+        <sensor name="camera_sensor" type="camera">
+            <pose>0 0 0 0 0 0</pose>
+            <visualize>true</visualize>
+            <update_rate>10.0</update_rate>
+            <plugin name="camera_controller" filename="libgazebo_ros_camera.so">
+                <!-- Set TF frame name. If empty, defaults to link name -->
+                <frame_name>camera_link</frame_name>
+            </plugin>
+        </sensor>
+    </gazebo>
 </robot>
